File: main/main.sch (KiCad schematic (older format))
At the start: 24 parts, among them J1 Conn_01x05, J2 Conn_02x32_Row_Letter_Last, U1 THS7374

Commit message: Add main PCB
Also some minor tweaks.
Parts:
- J1: footprint Connector_JST_NH:JST_NH_B5P-SHF-1AA_1x05_P2.50mm_Vertical -> Connector_JST_NH:JST_NH_BS5P-SHF-1AA_1x05_P2.50mm_Horizontal
Changed lines of the file:
@@
 F 0 "J1" H 1718 4217 50  0000 C CNN
 F 1 "Conn_01x05" H 1718 4126 50  0000 C CNN
-F 2 "Connector_JST_NH:JST_NH_B5P-SHF-1AA_1x05_P2.50mm_Vertical" H 1800 3800 50  0001 C CNN
+F 2 "Connector_JST_NH:JST_NH_BS5P-SHF-1AA_1x05_P2.50mm_Horizontal" H 1800 3800 50  0001 C CNN
 F 3 "~" H 1800 3800 50  0001 C CNN
 	1    1800 3800

Commit message: Use proper mounting holes rather than edge cuts
Parts:
- added H1, H2, H3, H4: MountingHole, MountingHole:MountingHole_3.2mm_M3, symbol Mechanical:MountingHole
Changed lines of the file:
@@
+	1    0    0    -1
+$EndComp
+$Comp
+L Mechanical:MountingHole H1
+U 1 1 634959A9
+P 5500 7350
+F 0 "H1" H 5600 7396 50  0000 L CNN
+F 1 "MountingHole" H 5600 7305 50  0000 L CNN
+F 2 "MountingHole:MountingHole_3.2mm_M3" H 5500 7350 50  0001 C CNN
+F 3 "~" H 5500 7350 50  0001 C CNN
+	1    5500 7350
+	1    0    0    -1
+$EndComp
+$Comp
+L Mechanical:MountingHole H2
+U 1 1 634959F3
+P 6250 7350
+F 0 "H2" H 6350 7396 50  0000 L CNN
+F 1 "MountingHole" H 6350 7305 50  0000 L CNN
+F 2 "MountingHole:MountingHole_3.2mm_M3" H 6250 7350 50  0001 C CNN
+F 3 "~" H 6250 7350 50  0001 C CNN
+	1    6250 7350
+	1    0    0    -1
+$EndComp
+$Comp
+L Mechanical:MountingHole H3
+U 1 1 63495DDE
+P 5500 7600
+F 0 "H3" H 5600 7646 50  0000 L CNN
+F 1 "MountingHole" H 5600 7555 50  0000 L CNN
+F 2 "MountingHole:MountingHole_3.2mm_M3" H 5500 7600 50  0001 C CNN
+F 3 "~" H 5500 7600 50  0001 C CNN
+	1    5500 7600
+	1    0    0    -1
+$EndComp
+$Comp
+L Mechanical:MountingHole H4
+U 1 1 634962A3
+P 6250 7600
+F 0 "H4" H 6350 7646 50  0000 L CNN
+F 1 "MountingHole" H 6350 7555 50  0000 L CNN
+F 2 "MountingHole:MountingHole_3.2mm_M3" H 6250 7600 50  0001 C CNN
+F 3 "~" H 6250 7600 50  0001 C CNN
+	1    6250 7600
 	1    0    0    -1
 $EndComp
