File: main/mcu.sch (KiCad schematic (older format))
At the start: 23 parts, among them J6 Conn_02x03_Odd_Even, Q3 DTC144EKA, SW2 PBSW_DPDT, U10 ATmega328PB-AU, U8 74LVC125, U9 arduino-nano-v3, Y1 Crystal_GND2

Commit message: Add main PCB
Also some minor tweaks.
Parts:
- Y1: footprint Crystal:Resonator_SMD_muRata_CSTxExxV-3Pin_3.0x1.1mm_HandSoldering -> Crystal:Resonator_SMD_muRata_CSTxExxV-3Pin_3.0x1.1mm
Changed lines of the file:
@@
 F 0 "Y1" V 10400 2500 50  0000 C CNN
 F 1 "Crystal_GND2" V 10300 2500 50  0000 C CNN
-F 2 "Crystal:Resonator_SMD_muRata_CSTxExxV-3Pin_3.0x1.1mm_HandSoldering" H 10200 3050 50  0001 C CNN
+F 2 "Crystal:Resonator_SMD_muRata_CSTxExxV-3Pin_3.0x1.1mm" H 10200 3050 50  0001 C CNN
 F 3 "~" H 10200 3050 50  0001 C CNN
 	1    10200 3050

Commit message: Change 74LVC125 to 74VHC125
This particular LVC part can't be used with a 5V supply. The single gate
LVC parts used elsewhere are fine.
Parts:
- U8: value 74LVC125 -> 74VHC125
Changed lines of the file:
@@
 P 2100 2400
 F 0 "U8" H 2100 2717 50  0000 C CNN
-F 1 "74LVC125" H 2100 2626 50  0000 C CNN
+F 1 "74VHC125" H 2100 2626 50  0000 C CNN
 F 2 "Package_SO:TSSOP-14_4.4x5mm_P0.65mm" H 2100 2400 50  0001 C CNN
 F 3 "http://www.ti.com/lit/gpn/sn74LVC125" H 2100 2400 50  0001 C CNN
@@
 P 2100 3200
 F 0 "U8" H 2100 3517 50  0000 C CNN
-F 1 "74LVC125" H 2100 3426 50  0000 C CNN
+F 1 "74VHC125" H 2100 3426 50  0000 C CNN
 F 2 "Package_SO:TSSOP-14_4.4x5mm_P0.65mm" H 2100 3200 50  0001 C CNN
 F 3 "http://www.ti.com/lit/gpn/sn74LVC125" H 2100 3200 50  0001 C CNN
@@
 P 2100 4000
 F 0 "U8" H 2100 4317 50  0000 C CNN
-F 1 "74LVC125" H 2100 4226 50  0000 C CNN
+F 1 "74VHC125" H 2100 4226 50  0000 C CNN
 F 2 "Package_SO:TSSOP-14_4.4x5mm_P0.65mm" H 2100 4000 50  0001 C CNN
 F 3 "http://www.ti.com/lit/gpn/sn74LVC125" H 2100 4000 50  0001 C CNN
@@
 P 2100 4800
 F 0 "U8" H 2100 5117 50  0000 C CNN
-F 1 "74LVC125" H 2100 5026 50  0000 C CNN
+F 1 "74VHC125" H 2100 5026 50  0000 C CNN
 F 2 "Package_SO:TSSOP-14_4.4x5mm_P0.65mm" H 2100 4800 50  0001 C CNN
 F 3 "http://www.ti.com/lit/gpn/sn74LVC125" H 2100 4800 50  0001 C CNN
@@
 P 3650 1450
 F 0 "U8" H 3880 1496 50  0000 L CNN
-F 1 "74LVC125" H 3880 1405 50  0000 L CNN
+F 1 "74VHC125" H 3880 1405 50  0000 L CNN
 F 2 "Package_SO:TSSOP-14_4.4x5mm_P0.65mm" H 3650 1450 50  0001 C CNN
 F 3 "http://www.ti.com/lit/gpn/sn74LVC125" H 3650 1450 50  0001 C CNN
